File: KINK-box.kicad_pcb (KiCad board)
At the start: 2 copper layers, 100 x 60 mm, 105 parts, among them J1 PJ-328A0-B, J2 QT02CSF83H0000G, J201 USB4500-03-0-A, J3 QT02CSF83H0000G, SW1 465M111172501, SW2 465M111172501, SW3 465M111172501, SW4 465M111172501, SW5 KMR223GLFG, U1 CH221K, U2 PCM5100A, U202 ESP32-S3-WROOM-1, U3 TPA3118D2DAPR, U4 BD33FC0FP, U5 P7805-2000R-S

Commit message: Fixed board edges
Parts:
- added H1: MountingHole_Pad, 0_NRD_footprints:ESP-solderhole, F.Cu at (66.2, 119.8)
Routing:
- net GND: track 34.7 -> 66.0 mm, vias 38 -> 85
- net +12V: track 157.3 -> 155.3 mm, vias 13 -> 12
- net /Logic/BTN2: track 18.2 -> 19.7 mm
- net +3V3: track 335.6 -> 336.6 mm
- net /Logic/I2S0_DATA: track 20.4 -> 19.7 mm
- net /Logic/BTN2_R: track 37.4 -> 36.8 mm
- net /Logic/BTN2_B: track 42.6 -> 42.1 mm
Other:
- outline, holes or cut-outs redrawn
- board text added: "KINK-box V1.0 @ Rvl"
- board text added: "Schematic based on Amped ESP32 by Sonocotta"
- board text added: "Solder fill here->"
- board text removed: "KINK-box V1.0 @ Rvl Schematic based on Amped ESP32 by Sonocotta"

Commit message: Fixed CH211 circuit and TPA3118D2 bugs
Parts:
- added C31: 2.2nF, Capacitor_SMD:C_0603_1608Metric, F.Cu at (74.8, 144.8)
- added C32: 2.2nF, Capacitor_SMD:C_0603_1608Metric, F.Cu at (83.0, 137.5)
- added R37: 5K1, Resistor_SMD:R_0603_1608Metric, F.Cu at (63.1, 138.9)
- added R41: 5K1, Resistor_SMD:R_0603_1608Metric, F.Cu at (65.0, 138.9)
- added R42: 5K1, Resistor_SMD:R_0603_1608Metric, F.Cu at (66.3, 133.6)
- added R43: 5K6, Resistor_SMD:R_0603_1608Metric, F.Cu at (115.0, 110.0)
- U5: value P7805-2000R-S -> P7803-2000R-S
- moved R1 2.67 mm to (68.6, 134.4)
- moved C14 1.60 mm to (117.0, 109.4)
Connections:
- C14 pad 1: +12V -> Net-(U3-GVDD)
- R1 pad 1: +12V -> Net-(U1-VDD)
- U1 pad 1: +12V -> Net-(U1-VDD)
- U202 pad 7: unconnected-(U202-GPIO7/TOUCH7/ADC1_CH6-Pad7) -> /Logic/~{PG}
- U3 pad 6: +12V -> Net-(U3-GVDD)
- U3 pad 7: GND -> Net-(U3-GVDD)
Routing:
- net /Logic/~{PG}: track 1.68 -> 18.7 mm
- net Net-(U3-GVDD): track 0.00 -> 14.4 mm, vias 0 -> 2
- net GND: track 66.0 -> 75.7 mm
- net +12V: track 155.3 -> 149.6 mm, vias 12 -> 10
- net Net-(U1-VDD): track 0.00 -> 5.24 mm
- net Net-(U3-GAIN/SLV): track 11.0 -> 14.0 mm
- net Net-(U1-CFG): track 2.07 -> 4.92 mm
- net Net-(C31-Pad2): track 29.4 -> 31.2 mm
- net Net-(C32-Pad2): track 21.1 -> 22.8 mm
- net Net-(J201-CC2): track 12.1 -> 13.0 mm
- net +3V3: track 336.6 -> 337.1 mm
Other:
- board text added: "KINK-box V1.1 @ RvL"
- board text removed: "KINK-box V1.0 @ Rvl"
