File: logic.kicad_sch (KiCad schematic)
At the start: 101 parts, among them J1 PJ-328A0-B, J2 QT02CSF83H0000G, J201 USB4500-03-0-A, J3 QT02CSF83H0000G, SW1 465M111172501, SW2 465M111172501, SW3 465M111172501, SW4 465M111172501, SW5 KMR223GLFG, U1 CH221K, U2 PCM5100A, U202 ESP32-S3-WROOM-1, U3 TPA3118D2DAPR, U4 BD33FC0FP, U5 P7805-2000R-S

Commit message: Fixed some meta-data
Other:
- company: (none) -> NURDspace
Changed lines of the file:
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@@
 		(date "2026-05-19")
 		(rev "V0.1.0")
+		(company "NURDspace")
 		(comment 1 "RvL")
 		(comment 2 "Schematic based on the Amped ESP32 by Sonocotta")

Commit message: Fixed CH211 circuit and TPA3118D2 bugs
Parts:
- added C31, C32: 2.2nF, Capacitor_SMD:C_0603_1608Metric, symbol 0_NRD_Capacitors_MLCC:C5_％＝_0603B222K500CT
- added R37, R41, R42: 5K1, Resistor_SMD:R_0603_1608Metric, symbol 0_NRD_Resistors:R_0603__5K1
- added R43: 5K6, Resistor_SMD:R_0603_1608Metric, symbol 0_NRD_Resistors:R_0603_5K6
- U5: value P7805-2000R-S -> P7803-2000R-S; S1 Description Non-Isolated DC/DC Converters 5 Vdc, 2 A, 10 W, 8 to 36 Vdc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 -> Non-Isolated DC/DC Converters 3.3 Vdc, 2 A, 10 W, 8 to 36 V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
Connections:
- net +12V: now also R42.1; no longer C14.1, R1.1, U1.1 (VDD), U3.6 (PLIMIT)
- net GND: now also C31.1, C32.1, R37.2, R41.2; no longer U3.7 (GVDD)
- net ~{PG}: now also U202.7 (GPIO7/TOUCH7/ADC1_CH6)
- net at J1.R, R5.2: now also C32.2
- net at J1.T, R4.2: now also C31.2
- net at R18.1, U3.8 (GAIN/SLV): now also R43.1
- net at J201.A5 (CC1), U1.4 (CC1): now also R37.1
- net at J201.B5 (CC2), U1.5 (CC2): now also R41.1
- new net: C14.1, R43.2, U3.6 (PLIMIT), U3.7 (GVDD)
- new net: R1.1, R42.2, U1.1 (VDD)
- no-connect marks 15 -> 14
Other:
- note added: "20dB gain"
- moved on the sheet: C1, J1, R18, R21
